File: accelerometre.kicad_sch (KiCad schematic)
At the start: 3 parts, among them J22 Conn_01x04_Socket

Commit message: V1GD
V1 20/10/25
Parts:
- R24, R25: footprint (none) -> Resistor_SMD:R_1206_3216Metric
Changed lines of the file:
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@@
 			)
 		)
-		(property "Footprint" ""
+		(property "Footprint" "Resistor_SMD:R_1206_3216Metric"
 			(at 109.728 71.12 90)
 			(effects
@@
 			)
 		)
-		(property "Footprint" ""
+		(property "Footprint" "Resistor_SMD:R_1206_3216Metric"
 			(at 99.568 71.12 90)
 			(effects
