File: power.kicad_sch (KiCad schematic)
At the start: 20 parts, among them J24 Conn_01x02_Socket, U2 LM2596S-ADJ, U3 LM2596S-ADJ

Commit message: V1GD
V1 20/10/25
Parts:
- C3, C6: value 220µF -> 470µF
- C5: value 180µF -> 470µF
- R17: value 2200 -> 4700
- R18, R19, R20, R21: footprint (none) -> Resistor_SMD:R_1206_3216Metric
Changed lines of the file:
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@@
 			)
 		)
-		(property "Value" "180µF"
+		(property "Value" "470µF"
 			(at 180.34 115.316 0)
 			(effects
@@
 			)
 		)
-		(property "Footprint" ""
+		(property "Footprint" "Resistor_SMD:R_1206_3216Metric"
 			(at 222.758 43.18 90)
 			(effects
@@
 			)
 		)
-		(property "Footprint" ""
+		(property "Footprint" "Resistor_SMD:R_1206_3216Metric"
 			(at 231.14 109.728 90)
 			(effects
@@
 			)
 		)
-		(property "Value" "220µF"
+		(property "Value" "470µF"
 			(at 251.46 111.7599 0)
 			(effects
@@
 			)
 		)
-		(property "Value" "220µF"
+		(property "Value" "470µF"
 			(at 250.19 58.4199 0)
 			(effects
@@
 			)
 		)
-		(property "Footprint" ""
+		(property "Footprint" "Resistor_SMD:R_1206_3216Metric"
 			(at 229.87 56.388 90)
 			(effects
@@
 			)
 		)
-		(property "Footprint" ""
+		(property "Footprint" "Resistor_SMD:R_1206_3216Metric"
 			(at 224.028 96.52 90)
 			(effects
@@
 			)
 		)
-		(property "Value" "2200"
+		(property "Value" "4700"
 			(at 144.78 76.2 90)
 			(effects
