File: rpipico.kicad_sch (KiCad schematic)
At the start: 1 part

Commit message: V1GD
V1 20/10/25
Parts:
- removed A1: RaspberryPi_Pico, Module:RaspberryPi_Pico_Common_Unspecified, symbol MCU_Module:RaspberryPi_Pico
- added A4: Arduino_UNO_R3, Module:Arduino_UNO_R3, symbol MCU_Module:Arduino_UNO_R3
Connections:
- net +3.3V: now also A4.4 (3V3)
- net +5V: now also A4.5 (+5V)
- net GND: now also A4.29 (GND), A4.6 (GND), A4.7 (GND)
- net UART0_RX: now also A4.15 (D0/RX)
- net UART0_TX: now also A4.16 (D1/TX)
- new net CM03: A4.12 (A3)
- new net CM04: A4.11 (A2)
- new net CM05: A4.10 (A1)
- new net CM06: A4.9 (A0)
- new net I2C0_SCL/CM01: A4.14 (SCL/A5)
- new net I2C0_SDA/CM02: A4.13 (SDA/A4)
- new net PWM1A: A4.18 (D3)
- new net PWM1B: A4.17 (D2)
- new net PWM2A: A4.20 (D5)
- new net PWM2B: A4.19 (D4)
- new net PWM3A: A4.21 (D6)
- new net PWM3B: A4.22 (D7)
- new net PWM4A: A4.24 (D9)
- new net PWM4B: A4.23 (D8)
- new net PWM5A: A4.25 (D10)
- new net PWM5B: A4.27 (D12)
- new net PWM6A: A4.26 (D11)
- new net PWM6B: A4.28 (D13)
- no-connect marks 5 -> 6
Other:
- note removed: "SPIx_SCK = SCK SPIx_TX = MOSI SPIx_RX = MISO"
