File: rpipico_zero.kicad_sch (KiCad schematic)
At the start: 0 parts

Commit message: V1GD
V1 20/10/25
Other:
- sheet Raspberry Pi Pico renamed arduino
- removed sheet Capteurs magnétiques AS5048a
- removed sheet Raspberry Pi Zero
- added sheet Raspberry Pi automate (rpizero.kicad_sch)
Changed lines of the file:
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@@
 	(paper "A4")
+	(sheet
+		(at 24.13 60.96)
+		(size 45.466 10.16)
+		(exclude_from_sim no)
+		(in_bom yes)
+		(on_board yes)
+		(dnp no)
+		(fields_autoplaced yes)
+		(stroke
+			(width 0.1524)
+			(type solid)
+		)
+		(fill
+			(color 0 0 0 0.0000)
+		)
+		(property "Sheetname" "Raspberry Pi automate"
+			(at 24.13 60.2484 0)
+			(effects
+				(font
+					(size 1.27 1.27)
+				)
+				(justify left bottom)
+			)
+		)
+		(property "Sheetfile" "rpizero.kicad_sch"
+			(at 24.13 71.7046 0)
+			(effects
+				(font
+					(size 1.27 1.27)
+				)
+				(justify left top)
+			)
+		)
+		(instances
+			(project "rpipico_zero"
+				(path "/867cba6c-c4f7-4f0e-b11e-bdca0b806b47"
+					(page "4")
+				)
+			)
+		)
+	)
 	(sheet
 		(at 24.638 79.502)
@@
 	)
 	(sheet
-		(at 24.892 97.282)
-		(size 45.466 10.16)
-		(exclude_from_sim no)
-		(in_bom yes)
-		(on_board yes)
-		(dnp no)
-		(fields_autoplaced yes)
-		(stroke
-			(width 0.1524)
-			(type solid)
-		)
-		(fill
-			(color 0 0 0 0.0000)
-		)
-		(property "Sheetname" "Raspberry Pi Zero"
-			(at 24.892 96.5704 0)
-			(effects
-				(font
-					(size 1.27 1.27)
-				)
-				(justify left bottom)
-			)
-		)
-		(property "Sheetfile" "rpizero.kicad_sch"
-			(at 24.892 108.0266 0)
-			(effects
-				(font
-					(size 1.27 1.27)
-				)
-				(justify left top)
-			)
-		)
-		(instances
-			(project "rpipico_zero"
-				(path "/867cba6c-c4f7-4f0e-b11e-bdca0b806b47"
-					(page "6")
-				)
-			)
-		)
-	)
-	(sheet
-		(at 25.146 180.594)
+		(at 24.384 163.068)
 		(size 45.466 9.144)
 		(exclude_from_sim no)
@@
 		)
 		(property "Sheetname" "Panneau LED"
-			(at 25.146 179.8824 0)
+			(at 24.384 162.3564 0)
 			(effects
 				(font
@@
 		)
 		(property "Sheetfile" "LED.kicad_sch"
-			(at 25.146 190.3226 0)
+			(at 24.384 172.7966 0)
 			(effects
 				(font
@@
 	)
 	(sheet
-		(at 25.146 165.1)
+		(at 24.384 147.574)
 		(size 45.466 9.652)
 		(exclude_from_sim no)
@@
 		)
 		(property "Sheetname" "Puissance"
-			(at 25.146 164.3884 0)
+			(at 24.384 146.8624 0)
 			(effects
 				(font
@@
 		)
 		(property "Sheetfile" "power.kicad_sch"
-			(at 25.146 175.3366 0)
+			(at 24.384 157.8106 0)
 			(effects
 				(font
@@
 	)
 	(sheet
-		(at 24.892 114.046)
+		(at 24.13 96.52)
 		(size 45.466 9.906)
 		(exclude_from_sim no)
@@
 		)
 		(property "Sheetname" "Capteurs de courant"
-			(at 24.892 113.3344 0)
+			(at 24.13 95.8084 0)
 			(effects
 				(font
@@
 		)
 		(property "Sheetfile" "Capteur_courant.kicad_sch"
-			(at 24.892 124.5366 0)
+			(at 24.13 107.0106 0)
 			(effects
 				(font
@@
 	)
 	(sheet
-		(at 24.384 61.214)
-		(size 45.72 10.16)
-		(exclude_from_sim no)
-		(in_bom yes)
-		(on_board yes)
-		(dnp no)
-		(fields_autoplaced yes)
-		(stroke
-			(width 0.1524)
-			(type solid)
-		)
-		(fill
-			(color 0 0 0 0.0000)
-		)
-		(property "Sheetname" "Capteurs magnétiques AS5048a"
-			(at 24.384 60.5024 0)
-			(effects
-				(font
-					(size 1.27 1.27)
-				)
-				(justify left bottom)
-			)
-		)
-		(property "Sheetfile" "as5048a.kicad_sch"
-			(at 24.384 71.9586 0)
-			(effects
-				(font
-					(size 1.27 1.27)
-				)
-				(justify left top)
-			)
-		)
-		(instances
-			(project "rpipico_zero"
-				(path "/867cba6c-c4f7-4f0e-b11e-bdca0b806b47"
-					(page "4")
-				)
-			)
-		)
-	)
-	(sheet
-		(at 25.146 148.59)
+		(at 24.384 131.064)
 		(size 45.466 10.16)
 		(exclude_from_sim no)
@@
 		)
 		(property "Sheetname" "Servo-moteur"
-			(at 25.146 147.8784 0)
+			(at 24.384 130.3524 0)
 			(effects
 				(font
@@
 		)
 		(property "Sheetfile" "servo.kicad_sch"
-			(at 25.146 159.3346 0)
+			(at 24.384 141.8086 0)
 			(effects
 				(font
@@
 			(color 0 0 0 0.0000)
 		)
-		(property "Sheetname" "Raspberry Pi Pico"
+		(property "Sheetname" "arduino"
 			(at 24.13 22.1484 0)
 			(effects
@@
 	)
 	(sheet
-		(at 25.146 131.064)
+		(at 24.384 113.538)
 		(size 45.212 10.414)
 		(exclude_from_sim no)
@@
 		)
 		(property "Sheetname" "Accéléromètre"
-			(at 25.146 130.3524 0)
+			(at 24.384 112.8264 0)
 			(effects
 				(font
@@
 		)
 		(property "Sheetfile" "accelerometre.kicad_sch"
-			(at 25.146 142.0626 0)
-			(effects
-				(font
+			(at 24.384 124.5366 0)
+			(effects
+				(font
